Commit message: modify orientation of lidar L1 and disable gazebo / ros2_control tags in urdf

File: urdf/go2_description.urdf (robot description, URDF)
Before this commit: robot go2_description, 29 links, 28 joints
Joints:
- joint radar_joint: origin xyz=0.28945 0 -0.046825 rpy=0 2.8782 0 -> xyz=0.28945 0 -0.046825 rpy=-2.913 -0.132 -1.057

File: urdf/go2_description.urdf.xacro (robot description, xacro)
@@ -113,4 +113,4 @@
   <xacro:go2_leg name="LR" x_joint="-0.1934" y_joint="0.0465" y_thigh_joint="0.0955"/>
   <xacro:go2_leg name="RR" x_joint="-0.1934" y_joint="-0.0465" y_thigh_joint="-0.0955"/>
-  <xacro:include filename="$(find go2_description)/urdf/gazebo.urdf.xacro"/>
+  <!-- <xacro:include filename="$(find go2_description)/urdf/gazebo.urdf.xacro"/> -->
 </robot>

File: urdf/leg.urdf.xacro (robot description, xacro)
@@ -157,5 +157,5 @@
       <axis xyz="0 0 0" />
     </joint>
-    <ros2_control name="${name}_control" type="system">
+    <!-- <ros2_control name="${name}_control" type="system">
       <hardware>
         <plugin>gazebo_ros2_control/GazeboSystem</plugin>
@@ -176,5 +176,5 @@
         <state_interface name="velocity"/>
       </joint>
-    </ros2_control>
+    </ros2_control>  -->
     <!-- <xacro:leg_transmission name="${name}"/> -->
   </xacro:macro>
