Commit message: Adding realsense and removing footprint

File: urdf/go2.urdf.xacro (robot description, xacro)
@@ -9,10 +9,3 @@
     <origin xyz="0.045 0 0.070" rpy="0 0 0"/>
   </xacro:sensor_d435i>
-  <!-- Base footprint -->
-  <link name="base_footprint" />
-  <joint name="base_footprint_joint" type="fixed">
-    <origin rpy="0 0 0" xyz="0 0 -0.37" />
-    <parent link="base_link" />
-    <child link="base_footprint" />
-  </joint>
 </robot>

Commit message: update some urdf files

File: urdf/go2.urdf.xacro (robot description, xacro)
@@ -6,5 +6,5 @@
   <xacro:arg name="use_nominal_extrinsics" default="false" />
   <xacro:include filename="$(find realsense2_description)/urdf/_d435i.urdf.xacro"/>
-  <xacro:sensor_d435i parent="Head_upper" use_nominal_extrinsics="$(arg use_nominal_extrinsics)">
+  <xacro:sensor_d435i parent="Head_upper" name="head_camera" use_nominal_extrinsics="$(arg use_nominal_extrinsics)">
     <origin xyz="0.045 0 0.070" rpy="0 0 0"/>
   </xacro:sensor_d435i>

File: urdf/go2_description.urdf.xacro (robot description, xacro)
@@ -15,5 +15,5 @@
       <origin xyz="0 0 0" rpy="0 0 0" />
       <geometry>
-         <mesh filename="file://$(find go2_description)/dae/base.dae" scale="1 1 1"/>
+         <mesh filename="package://go2_description/dae/base.dae" scale="1 1 1"/>
       </geometry>
       <material
