Commit message: Added Go2 gzsim. Copying from our unitree_ros fork

File: urdf/gazebo.urdf.xacro (robot description, xacro)
@@ -1,5 +1,5 @@
 <?xml version="1.0"?>
 <robot>
-    <gazebo>
+    <!--<gazebo>
       <plugin name="p3d_base_controller" filename="libgazebo_ros_p3d.so">
         <ros>
@@ -13,7 +13,7 @@
         <gaussian_noise>0.01</gaussian_noise>
     </plugin>
-    </gazebo>
+    </gazebo>-->
     <gazebo>
-        <plugin filename="libgazebo_ros2_control.so" name="gazebo_ros2_control">
+        <plugin filename="gz_ros2_control-system" name="gz_ros2_control::GazeboSimROS2ControlPlugin">
         <parameters>$(find go2_description)/config/ros_control/ros_control.yaml</parameters>
       </plugin>

File: urdf/go2_description.urdf.xacro (robot description, xacro)
@@ -1,22 +1,30 @@
 <?xml version="1.0"?>
 <robot xmlns:xacro="http://wiki.ros.org/xacro" name="go2">
-  <xacro:arg name="prefix" default=""/>
-  <xacro:include filename="$(find go2_description)/urdf/leg.urdf.xacro"/>
-<!-- Links -->
- <link name="base_link">
-    <inertial>
-      <origin xyz="0.021112 0 -0.005366" rpy="0 0 0" />
-      <mass value="6.921" />
-      <inertia
-        ixx="0.02448" ixy="0.00012166" ixz="0.0014849"
-        iyy="0.098077" iyz="-3.12E-05" izz="0.107" />
-    </inertial>
-    <visual>
-      <origin xyz="0 0 0" rpy="0 0 0" />
-      <geometry>
-         <mesh filename="package://go2_description/dae/base.dae" scale="1 1 1"/>
-      </geometry>
-      <material
-        name="">
+  <xacro:macro name="go2" params="mode">
+    <xacro:arg name="DEBUG" default="false"/>
+    <xacro:arg name="prefix" default=""/>
+    <xacro:include filename="$(find go2_description)/xacro/const.xacro"/>
+    <xacro:include filename="$(find go2_description)/xacro/materials.xacro"/>
+    <xacro:include filename="$(find go2_description)/xacro/leg.xacro"/>
+    <xacro:if value="${mode == 'gazebo'}">
+      <xacro:include filename="$(find go2_description)/xacro/gazebo.xacro"/>
+      <xacro:include filename="$(find go2_description)/xacro/camera_simulation.xacro"/>
+      <xacro:include filename="$(find go2_description)/xacro/ros2_control_macro.xacro"/>
+    </xacro:if>
+    <!-- Links -->
+    <link name="base_link">
+      <inertial>
+        <origin xyz="0.021112 0 -0.005366" rpy="0 0 0" />
+        <mass value="6.921" />
+        <inertia
+          ixx="0.02448" ixy="0.00012166" ixz="0.0014849"
+          iyy="0.098077" iyz="-3.12E-05" izz="0.107" />
+      </inertial>
+      <visual>
+        <origin xyz="0 0 0" rpy="0 0 0" />
+        <geometry>
+          <mesh filename="package://go2_description/dae/base.dae" scale="1 1 1"/>
+        </geometry>
+        <material name="">
         <color rgba="1 1 1 1" />
       </material>
@@ -28,7 +36,4 @@
       </geometry>
     </collision>
-  </link>
-  <link
-    name="odom">
   </link>
   <link name="Head_upper">
@@ -80,9 +85,4 @@
     </inertial>
   </link>
-  <joint name="odom_joint" type="fixed">
-    <origin xyz="0 0 0" rpy="0 0 0" />
-    <parent link="odom" />
-    <child link="base_link" />
-  </joint>
   <joint name="Head_upper_joint" type="fixed" dont_collapse="true">
     <origin xyz="0.285 0 0.01" rpy="0 0 0" />
@@ -104,13 +104,29 @@
   </joint>
   <joint name="radar_joint" type="fixed">
-    <origin xyz="0.28945 0 -0.046825" rpy="0 2.8782 0" />
+    <origin xyz="0.28945 0 -0.046825" rpy="-2.913 -0.132 -1.057" />
     <parent link="base_link" />
     <child link="radar" />
     <axis xyz="0 0 0" />
   </joint>
-  <xacro:go2_leg name="LF" x_joint="0.1934" y_joint="0.0465" y_thigh_joint="0.0955"/>
-  <xacro:go2_leg name="RF" x_joint="0.1934" y_joint="-0.0465" y_thigh_joint="-0.0955"/>
-  <xacro:go2_leg name="LR" x_joint="-0.1934" y_joint="0.0465" y_thigh_joint="0.0955"/>
-  <xacro:go2_leg name="RR" x_joint="-0.1934" y_joint="-0.0465" y_thigh_joint="-0.0955"/>
-  <!-- <xacro:include filename="$(find go2_description)/urdf/gazebo.urdf.xacro"/> -->
+    <xacro:leg name="FR" mirror="-1" mirror_dae= "False" front_hind="1"  front_hind_dae="True"  />
+    <xacro:leg name="FL" mirror="1"  mirror_dae="True"   front_hind="1"  front_hind_dae="True"  />
+    <xacro:leg name="RR" mirror="-1" mirror_dae="False"  front_hind="-1" front_hind_dae="False" />
+    <xacro:leg name="RL" mirror="1"  mirror_dae="True"   front_hind="-1" front_hind_dae="False" />
+    <xacro:if value="${mode == 'gazebo'}">
+            <xacro:go2_ros2_control interface_type="gazebo"/>
+                <!-- PosePublisher - P3D-equivalent -->
+            <xacro:macro name="go2_pose_publisher">
+            <gazebo>
+                <plugin filename="gz-sim-pose-publisher-system" name="gz::sim::systems::PosePublisher">
+                <publish_link_pose>false</publish_link_pose>
+                <publish_nested_model_pose>true</publish_nested_model_pose>
+                <publish_model_pose>true</publish_model_pose>
+                <update_frequency>30</update_frequency>
+                <use_pose_vector_msg>false</use_pose_vector_msg>
+                </plugin>
+            </gazebo>
+            </xacro:macro>
+            <xacro:go2_pose_publisher />
+    </xacro:if>
+  </xacro:macro>
 </robot>

File: xacro/gazebo.xacro (robot description, xacro)
@@ -3,8 +3,7 @@
     <!-- ros_control plugin -->
     <gazebo>
-        <plugin name="gazebo_ros_control" filename="libgazebo_ros_control.so">
-            <robotNamespace>/go2_gazebo</robotNamespace>
-            <robotSimType>gazebo_ros_control/DefaultRobotHWSim</robotSimType>
-        </plugin>
+      <plugin name="gz_ros2_control::GazeboSimROS2ControlPlugin" filename="gz_ros2_control-system">
+        <parameters>$(find go2_description)/config/ros_control/ros_control_gazebo.yaml</parameters>
+      </plugin>
     </gazebo>
     <!-- Show the trajectory of trunk center. -->
@@ -18,7 +17,7 @@
             </plot>
         </plugin>
-    </gazebo-->
+    </gazebo>-->
     <!-- Show the trajectory of foot. You can add another trajectory about another foot. -->
-     <gazebo>
+     <!--<gazebo>
         <plugin name="3dplot" filename="libLinkPlot3DPlugin.so">
             <frequency>100</frequency>
@@ -34,5 +33,5 @@
             <topicName>/apply_force/trunk</topicName>
         </plugin>
-    </gazebo>
+    </gazebo>-->
     <gazebo reference="imu_link">
         <gravity>true</gravity>
@@ -42,5 +41,5 @@
             <visualize>true</visualize>
             <topic>__default_topic__</topic>
-            <plugin filename="libgazebo_ros_imu_sensor.so" name="imu_plugin">
+            <plugin filename="gz-sim-imu-system" name="gz::sim::systems::Imu">
                 <topicName>trunk_imu</topicName>
                 <bodyName>imu_link</bodyName>
@@ -55,5 +54,5 @@
     </gazebo>
     <!-- Foot contacts. -->
-    <gazebo reference="FR_calf">
+    <!--<gazebo reference="FR_calf">
         <sensor name="FR_foot_contact" type="contact">
         <update_rate>100</update_rate>
@@ -90,7 +89,7 @@
         </contact>
         </sensor>
-    </gazebo>
+    </gazebo>-->
     <!-- Visualization of Foot contacts. -->
-    <gazebo reference="FR_foot">
+    <!--<gazebo reference="FR_foot">
         <visual>
             <plugin name="drawForcePlugin" filename="libunitreeDrawForcePlugin.so">
@@ -119,5 +118,5 @@
             </plugin>
         </visual>
-    </gazebo>
+    </gazebo>-->
     <gazebo reference="base">
         <turnGravityOff>false</turnGravityOff>

File: xacro/leg.xacro (robot description, xacro)
@@ -16,5 +16,5 @@
                 <origin rpy="0 0 0" xyz="${-leg_offset_x} ${leg_offset_y} 0"/>
             </xacro:if>
-            <parent link="trunk"/>
+            <parent link="base_link"/>
             <child link="${name}_hip"/>
             <axis xyz="1 0 0"/>

File: xacro/robot.urdf.xacro (robot description, xacro)
@@ -1,7 +1,8 @@
 <?xml version="1.0"?>
-<robot name="go2" xmlns:xacro="http://www.ros.org/wiki/xacro">
+<robot xmlns:xacro="http://wiki.ros.org/xacro" name="go2">
+  <xacro:arg name="mode" default="gazebo"/>
   <!-- Go2 -->
-  <xacro:include filename="$(find go2_description)/urdf/go2_description.urdf.xacro" />
-  <xacro:go2 mode="gazebo"/>
+  <xacro:include filename="$(find go2_description)/urdf/go2_description.urdf.xacro"/>
+  <xacro:go2 mode="$(arg mode)"/>
   <!-- Realsense D435i -->
   <xacro:arg name="use_nominal_extrinsics" default="false" />

File: xacro/robot.xacro (robot description, xacro)
@@ -1,113 +1,141 @@
 <?xml version="1.0"?>
 <robot name="go2" xmlns:xacro="http://www.ros.org/wiki/xacro">
-    <xacro:arg name="DEBUG" default="false"/>
-    <xacro:include filename="$(find go2_description)/xacro/const.xacro"/>
-    <xacro:include filename="$(find go2_description)/xacro/materials.xacro"/>
-    <xacro:include filename="$(find go2_description)/xacro/leg.xacro"/>
-    <!-- <xacro:include filename="$(find go2_description)/xacro/stairs.xacro"/> -->
-    <xacro:include filename="$(find go2_description)/xacro/gazebo.xacro"/>
-    <!-- <xacro:include filename="$(find go2_gazebo)/launch/stairs.urdf.xacro"/> -->
-    <!-- <xacro:stairs stairs="15" xpos="0" ypos="0" zpos="0" /> -->
-    <!-- Rotor related joint and link is only for demonstrate location. -->
-    <!-- Actually, the rotor will rotate and the joint is not fixed. Reduction ratio should be considered. -->
-    <!-- Debug mode will hung up the robot, use "true" or "false" to switch it. -->
-    <xacro:if value="$(arg DEBUG)">
-        <link name="world"/>
-        <joint name="base_static_joint" type="fixed">
+    <xacro:macro name="go2" params="mode">
+        <xacro:arg name="DEBUG" default="false"/>
+        <xacro:include filename="$(find go2_description)/xacro/const.xacro"/>
+        <xacro:include filename="$(find go2_description)/xacro/materials.xacro"/>
+        <xacro:include filename="$(find go2_description)/xacro/leg.xacro"/>
+        <!-- <xacro:include filename="$(find go2_description)/xacro/stairs.xacro"/> -->
+        <xacro:if value="${mode == 'gazebo'}">
+            <xacro:include filename="$(find go2_description)/xacro/gazebo.xacro"/>
+            <xacro:include filename="$(find go2_description)/xacro/ros2_control_macro.xacro"/>
+        </xacro:if>
+        <!-- <xacro:include filename="$(find go2_gazebo)/launch/stairs.urdf.xacro"/> -->
+        <!-- <xacro:stairs stairs="15" xpos="0" ypos="0" zpos="0" /> -->
+        <!-- Rotor related joint and link is only for demonstrate location. -->
+        <!-- Actually, the rotor will rotate and the joint is not fixed. Reduction ratio should be considered. -->
+        <!-- Debug mode will hung up the robot, use "true" or "false" to switch it. -->
+        <xacro:if value="$(arg DEBUG)">
+            <link name="world"/>
+            <joint name="base_static_joint" type="fixed">
+                <origin rpy="0 0 0" xyz="0 0 0"/>
+                <parent link="world"/>
+                <child link="base"/>
+            </joint>
+        </xacro:if>
+        <link name="base">
+            <visual>
+                <origin rpy="0 0 0" xyz="0 0 0"/>
+                <geometry>
+                    <box size="0.001 0.001 0.001"/>
+                </geometry>
+            </visual>
+        </link>
+        <joint name="floating_base" type="fixed">
             <origin rpy="0 0 0" xyz="0 0 0"/>
-            <parent link="world"/>
-            <child link="base"/>
+            <parent link="base"/>
+            <child link="trunk"/>
         </joint>
-    </xacro:if>
-    <link name="base">
-        <visual>
+        <link name="trunk">
+            <visual>
+                <origin rpy="0 0 0" xyz="0 0 0"/>
+                <geometry>
+                    <mesh filename="package://go2_description/meshes/trunk.dae" scale="1 1 1"/>
+                </geometry>
+                <!-- <material name="orange"/> -->
+            </visual>
+            <collision>
+                <origin rpy="0 0 0" xyz="0 0 0"/>
+                <geometry>
+                    <box size="${trunk_length} ${trunk_width} ${trunk_height}"/>
+                </geometry>
+            </collision>
+            <inertial>
+                <origin rpy="0 0 0" xyz="${trunk_com_x} ${trunk_com_y} ${trunk_com_z}"/>
+                <mass value="${trunk_mass}"/>
+                <inertia
+                    ixx="${trunk_ixx}" ixy="${trunk_ixy}" ixz="${trunk_ixz}"
+                    iyy="${trunk_iyy}" iyz="${trunk_iyz}"
+                    izz="${trunk_izz}"/>
+            </inertial>
+        </link>
+        <joint name="imu_joint" type="fixed">
+            <parent link="trunk"/>
+            <child link="imu_link"/>
             <origin rpy="0 0 0" xyz="0 0 0"/>
-            <geometry>
-                <box size="0.001 0.001 0.001"/>
-            </geometry>
-        </visual>
-    </link>
-    <joint name="floating_base" type="fixed">
-        <origin rpy="0 0 0" xyz="0 0 0"/>
-        <parent link="base"/>
-        <child link="trunk"/>
-    </joint>
-    <link name="trunk">
-        <visual>
+        </joint>
+        <link name="imu_link">
+            <inertial>
+                <mass value="0.001"/>
+                <origin rpy="0 0 0" xyz="0 0 0"/>
+                <inertia ixx="0.0001" ixy="0" ixz="0" iyy="0.0001" iyz="0" izz="0.0001"/>
+            </inertial>
+            <visual>
+                <origin rpy="0 0 0" xyz="0 0 0"/>
+                <geometry>
+                    <box size="0.001 0.001 0.001"/>
+                </geometry>
+                <!-- <material name="red"/> -->
+            </visual>
+            <collision>
+                <origin rpy="0 0 0" xyz="0 0 0"/>
+                <geometry>
+                    <box size=".001 .001 .001"/>
+                </geometry>
+            </collision>
+        </link>
+        <joint name="front_camera_joint" type="fixed">
+            <parent link="trunk"/>
+            <child link="front_camera"/>
+            <origin rpy="0 0 0" xyz="0.32715 -0.00003 0.04297"/>
+        </joint>
+        <link name="front_camera">
+        </link>
+        <!--
+        <joint name="load_joint" type="fixed">
+            <parent link="trunk"/>
+            <child link="load_link"/>
             <origin rpy="0 0 0" xyz="0 0 0"/>
-            <geometry>
-                <mesh filename="package://go2_description/meshes/trunk.dae" scale="1 1 1"/>
-            </geometry>
-            <!-- <material name="orange"/> -->
-        </visual>
-        <collision>
-            <origin rpy="0 0 0" xyz="0 0 0"/>
-            <geometry>
-                <box size="${trunk_length} ${trunk_width} ${trunk_height}"/>
-            </geometry>
-        </collision>
-        <inertial>
-            <origin rpy="0 0 0" xyz="${trunk_com_x} ${trunk_com_y} ${trunk_com_z}"/>
-            <mass value="${trunk_mass}"/>
-            <inertia
-                ixx="${trunk_ixx}" ixy="${trunk_ixy}" ixz="${trunk_ixz}"
-                iyy="${trunk_iyy}" iyz="${trunk_iyz}"
-                izz="${trunk_izz}"/>
-        </inertial>
-    </link>
-    <joint name="imu_joint" type="fixed">
-        <parent link="trunk"/>
-        <child link="imu_link"/>
-        <origin rpy="0 0 0" xyz="0 0 0"/>
-    </joint>
-    <link name="imu_link">
-        <inertial>
-            <mass value="0.001"/>
-            <origin rpy="0 0 0" xyz="0 0 0"/>
-            <inertia ixx="0.0001" ixy="0" ixz="0" iyy="0.0001" iyz="0" izz="0.0001"/>
-        </inertial>
-        <visual>
-            <origin rpy="0 0 0" xyz="0 0 0"/>
-            <geometry>
-                <box size="0.001 0.001 0.001"/>
-            </geometry>
-            <!-- <material name="red"/> -->
-        </visual>
-        <collision>
-            <origin rpy="0 0 0" xyz="0 0 0"/>
-            <geometry>
-                <box size=".001 .001 .001"/>
-            </geometry>
-        </collision>
-    </link>
-    <!--
-    <joint name="load_joint" type="fixed">
-        <parent link="trunk"/>
-        <child link="load_link"/>
-        <origin rpy="0 0 0" xyz="0 0 0"/>
-    </joint>
-    <link name="load_link">
-        <inertial>
-            <mass value="5"/>
-            <origin rpy="0 0 0" xyz="0 0 0"/>
-            <inertia ixx="0.01" ixy="0" ixz="0" iyy="0.01" iyz="0" izz="0.01"/>
-        </inertial>
-        <visual>
-            <origin rpy="0 0 0" xyz="0 0 0.2"/>
-            <geometry>
-                <box size="0.5 0.3 0.2"/>
-            </geometry>
-        </visual>
-        <collision>
-            <origin rpy="0 0 0" xyz="0 0 0"/>
-            <geometry>
-                <box size=".001 .001 .001"/>
-            </geometry>
-        </collision>
-    </link>
--->
-    <xacro:leg name="FR" mirror="-1" mirror_dae= "False" front_hind="1"  front_hind_dae="True"  />
-    <xacro:leg name="FL" mirror="1"  mirror_dae="True"   front_hind="1"  front_hind_dae="True"  />
-    <xacro:leg name="RR" mirror="-1" mirror_dae="False"  front_hind="-1" front_hind_dae="False" />
-    <xacro:leg name="RL" mirror="1"  mirror_dae="True"   front_hind="-1" front_hind_dae="False" />
+        </joint>
+        <link name="load_link">
+            <inertial>
+                <mass value="5"/>
+                <origin rpy="0 0 0" xyz="0 0 0"/>
+                <inertia ixx="0.01" ixy="0" ixz="0" iyy="0.01" iyz="0" izz="0.01"/>
+            </inertial>
+            <visual>
+                <origin rpy="0 0 0" xyz="0 0 0.2"/>
+                <geometry>
+                    <box size="0.5 0.3 0.2"/>
+                </geometry>
+            </visual>
+            <collision>
+                <origin rpy="0 0 0" xyz="0 0 0"/>
+                <geometry>
+                    <box size=".001 .001 .001"/>
+                </geometry>
+            </collision>
+        </link>
+    -->
+        <xacro:leg name="FR" mirror="-1" mirror_dae= "False" front_hind="1"  front_hind_dae="True"  />
+        <xacro:leg name="FL" mirror="1"  mirror_dae="True"   front_hind="1"  front_hind_dae="True"  />
+        <xacro:leg name="RR" mirror="-1" mirror_dae="False"  front_hind="-1" front_hind_dae="False" />
+        <xacro:leg name="RL" mirror="1"  mirror_dae="True"   front_hind="-1" front_hind_dae="False" />
+        <xacro:if value="${mode == 'gazebo'}">
+            <xacro:go2_ros2_control interface_type="gazebo"/>
+                <!-- PosePublisher - P3D-equivalent -->
+            <xacro:macro name="go2_pose_publisher">
+            <gazebo>
+                <plugin filename="gz-sim-pose-publisher-system" name="gz::sim::systems::PosePublisher">
+                <publish_link_pose>false</publish_link_pose>
+                <publish_nested_model_pose>true</publish_nested_model_pose>
+                <publish_model_pose>true</publish_model_pose>
+                <update_frequency>30</update_frequency>
+                <use_pose_vector_msg>false</use_pose_vector_msg>
+                </plugin>
+            </gazebo>
+            </xacro:macro>
+            <xacro:go2_pose_publisher />
+        </xacro:if>
+    </xacro:macro>
 </robot>
