Commit message: fix go2 simulation

File: urdf/gazebo.urdf.xacro (robot description, xacro)
@@ -1,5 +1,5 @@
 <?xml version="1.0"?>
 <robot>
-    <gazebo>
+    <!-- <gazebo>
       <plugin name="p3d_base_controller" filename="libgazebo_ros_p3d.so">
         <ros>
@@ -13,9 +13,13 @@
         <gaussian_noise>0.01</gaussian_noise>
     </plugin>
-    </gazebo>
+    </gazebo> -->
     <gazebo>
-        <plugin filename="libgazebo_ros2_control.so" name="gazebo_ros2_control">
+        <!-- <plugin filename="libgazebo_ros2_control.so" name="gazebo_ros2_control">
         <parameters>$(find go2_description)/config/ros_control/ros_control.yaml</parameters>
-      </plugin>
+      </plugin> -->
+      <plugin name="gz_ros2_control::GazeboSimROS2ControlPlugin" filename="gz_ros2_control-system">
+        <parameters>$(find go2_description)/config/ros_control/ros2_control_go2.yaml</parameters>
+        <!-- <parameters>$(find go2_description)/config/ros_control/ros_control.yaml</parameters> -->
+    </plugin>
     </gazebo>
     <gazebo reference="base_link">

File: urdf/go2.urdf.xacro (robot description, xacro)
@@ -2,5 +2,5 @@
 <robot name="go2" xmlns:xacro="http://www.ros.org/wiki/xacro">
   <!-- Go2 -->
-  <xacro:include filename="$(find go2_description)/urdf/go2_description.urdf" />
+  <xacro:include filename="$(find go2_description)/urdf/go2_description.urdf.xacro" />
   <!-- Realsense D435i -->
   <xacro:arg name="use_nominal_extrinsics" default="false" />

File: urdf/go2_description.urdf.xacro (robot description, xacro)
@@ -1,8 +1,10 @@
 <?xml version="1.0"?>
 <robot xmlns:xacro="http://wiki.ros.org/xacro" name="go2">
-  <xacro:arg name="prefix" default=""/>
-  <xacro:include filename="$(find go2_description)/urdf/leg.urdf.xacro"/>
-<!-- Links -->
- <link name="base_link">
+  <xacro:arg name="prefix" default="" />
+  <xacro:include filename="$(find go2_description)/xacro/const.xacro"/>
+  <xacro:include filename="$(find go2_description)/xacro/materials.xacro"/>
+  <xacro:include filename="$(find go2_description)/urdf/leg.urdf.xacro" />
+  <!-- Links -->
+  <link name="base_link">
     <inertial>
       <origin xyz="0.021112 0 -0.005366" rpy="0 0 0" />
@@ -15,5 +17,5 @@
       <origin xyz="0 0 0" rpy="0 0 0" />
       <geometry>
-         <mesh filename="package://go2_description/dae/base.dae" scale="1 1 1"/>
+        <mesh filename="package://go2_description/dae/base.dae" scale="1 1 1" />
       </geometry>
       <material
@@ -28,7 +30,4 @@
       </geometry>
     </collision>
-  </link>
-  <link
-    name="odom">
   </link>
   <link name="Head_upper">
@@ -80,9 +79,4 @@
     </inertial>
   </link>
-  <joint name="odom_joint" type="fixed">
-    <origin xyz="0 0 0" rpy="0 0 0" />
-    <parent link="odom" />
-    <child link="base_link" />
-  </joint>
   <joint name="Head_upper_joint" type="fixed" dont_collapse="true">
     <origin xyz="0.285 0 0.01" rpy="0 0 0" />
@@ -91,5 +85,5 @@
     <axis xyz="0 0 0" />
   </joint>
- <joint name="Head_lower_joint" type="fixed" dont_collapse="true">
+  <joint name="Head_lower_joint" type="fixed" dont_collapse="true">
     <origin xyz="0.008 0 -0.07" rpy="0 0 0" />
     <parent link="Head_upper" />
@@ -109,8 +103,23 @@
     <axis xyz="0 0 0" />
   </joint>
-  <xacro:go2_leg name="LF" x_joint="0.1934" y_joint="0.0465" y_thigh_joint="0.0955"/>
-  <xacro:go2_leg name="RF" x_joint="0.1934" y_joint="-0.0465" y_thigh_joint="-0.0955"/>
-  <xacro:go2_leg name="LR" x_joint="-0.1934" y_joint="0.0465" y_thigh_joint="0.0955"/>
-  <xacro:go2_leg name="RR" x_joint="-0.1934" y_joint="-0.0465" y_thigh_joint="-0.0955"/>
-  <!-- <xacro:include filename="$(find go2_description)/urdf/gazebo.urdf.xacro"/> -->
+  <xacro:go2_leg name="LF" x_joint="0.1934" y_joint="0.0465" y_thigh_joint="0.0955" />
+  <xacro:go2_leg name="RF" x_joint="0.1934" y_joint="-0.0465" y_thigh_joint="-0.0955" />
+  <xacro:go2_leg name="LR" x_joint="-0.1934" y_joint="0.0465" y_thigh_joint="0.0955" />
+  <xacro:go2_leg name="RR" x_joint="-0.1934" y_joint="-0.0465" y_thigh_joint="-0.0955" />
+  <xacro:include filename="$(find go2_description)/urdf/gazebo.urdf.xacro" />
+  <xacro:include filename="$(find go2_description)/urdf/ros2_control_macro.xacro" />
+  <xacro:go2_ros2_control interface_type="gazebo" />
+  <!-- PosePublisher - P3D-equivalent -->
+  <xacro:macro name="go2_pose_publisher">
+    <gazebo>
+      <plugin filename="gz-sim-pose-publisher-system" name="gz::sim::systems::PosePublisher">
+        <publish_link_pose>false</publish_link_pose>
+        <publish_nested_model_pose>true</publish_nested_model_pose>
+        <publish_model_pose>true</publish_model_pose>
+        <update_frequency>30</update_frequency>
+        <use_pose_vector_msg>false</use_pose_vector_msg>
+      </plugin>
+    </gazebo>
+  </xacro:macro>
+  <xacro:go2_pose_publisher />
 </robot>

File: urdf/leg.urdf.xacro (robot description, xacro)
@@ -2,5 +2,5 @@
 <robot xmlns:xacro="http://ros.org/wiki/xacro">
   <xacro:macro name="go2_leg" params="name  x_joint y_joint y_thigh_joint" >
-    <!-- <xacro:include filename="$(find go2_description)/urdf/transmission.urdf.xacro"/> -->
+    <xacro:include filename="$(find go2_description)/urdf/transmission.urdf.xacro"/>
     <xacro:property name="LF" value="LF" />
     <xacro:property name="RF" value="RF" />
@@ -159,7 +159,8 @@
     <!-- <ros2_control name="${name}_control" type="system">
       <hardware>
-        <plugin>gazebo_ros2_control/GazeboSystem</plugin>
+        <plugin>gz_ros2_control/GazeboSimSystem</plugin>
       </hardware>
       <joint name="${name}_hip_joint">
+        <command_interface name="position"/>
         <command_interface name="effort"/>
         <state_interface name="position"/>
@@ -167,4 +168,5 @@
       </joint>
       <joint name="${name}_upper_leg_joint">
+        <command_interface name="position"/>
         <command_interface name="effort"/>
         <state_interface name="position"/>
@@ -172,10 +174,11 @@
       </joint>
       <joint name="${name}_lower_leg_joint">
+        <command_interface name="position"/>
         <command_interface name="effort"/>
         <state_interface name="position"/>
         <state_interface name="velocity"/>
       </joint>
-    </ros2_control>  -->
-    <!-- <xacro:leg_transmission name="${name}"/> -->
+    </ros2_control> -->
+    <xacro:leg_transmission name="${name}"/>
   </xacro:macro>
 </robot>

File: xacro/gazebo.xacro (robot description, xacro)
@@ -3,7 +3,10 @@
     <!-- ros_control plugin -->
     <gazebo>
-        <plugin name="gazebo_ros_control" filename="libgazebo_ros_control.so">
+        <!-- <plugin name="gazebo_ros_control" filename="libgazebo_ros_control.so">
             <robotNamespace>/go2_gazebo</robotNamespace>
             <robotSimType>gazebo_ros_control/DefaultRobotHWSim</robotSimType>
+        </plugin> -->
+        <plugin name="gz_ros2_control::GazeboSimROS2ControlPlugin" filename="gz_ros2_control-system">
+            <parameters>$(find go2_description)/config/ros2_control_go2.yaml</parameters>
         </plugin>
     </gazebo>
